File: stm32_imu.kicad_sch (KiCad schematic)
At the start: 44 parts, among them J1 USB_C_Receptacle_USB2.0_16P, J3 TC2030, U1 NRF24L01, U3 LM1117MP-3.3, U4 2.4GHz, U5 ICM-20948, U6 STM32F411CEUx, Y1 16MHz, Y2 24MHz

Commit message: Add files via upload
Parts:
- removed D2, D3: ESD, Diode_SMD:D_SOD-923, symbol Device:D_TVS
- added U2: USBLC6-2SC6, Package_TO_SOT_SMD:SOT-23-6, symbol Power_Protection:USBLC6-2SC6
- C12, C13, C14, C15, C16, C17, C18, C20, C21, C22, C23, C24: footprint Capacitor_SMD:C_0201_0603Metric -> Capacitor_SMD:C_0402_1005Metric
- C19: footprint Capacitor_SMD:C_0402_1005Metric -> Capacitor_SMD:C_0603_1608Metric
- C4, C7: value 22u -> 10u; footprint Capacitor_SMD:C_0402_1005Metric -> Capacitor_SMD:C_0603_1608Metric
- FB1: value 600 @ 100MHz -> 100 @ 100MHz
Connections:
- net +3.3V: now also C7.1, U3.2 (VO); no longer FB1.2
- net CE: now also U6.19 (PB1); no longer U6.14 (PA4)
- net D+: now also U2.4 (I/O2); no longer J1.A6 (D+), J1.B6 (D+)
- net D-: now also U2.6 (I/O1); no longer J1.A7 (D-), J1.B7 (D-)
- net GND: now also U2.2 (GND); no longer J1.S1 (SHIELD)
- net IRQ: now also U6.14 (PA4); no longer U6.19 (PB1)
- net SPI1_MISO: no longer U5.24 (SDA/SDI)
- net SPI1_MOSI: no longer U5.9 (SDO/AD0)
- net SPI1_SCK: no longer U5.23 (SCL/SCLK)
- net VBUS: now also FB1.1, U2.5 (VBUS); no longer C4.1, U3.3 (VI)
- net SPI2_CS: now reaches U6.25 (PB12)
- net SPI2_CS: now also U5.22 (~{CS})
- net SPI2_SCK: now reaches U6.26 (PB13)
- net SPI2_SCK: now also U5.23 (SCL/SCLK)
- net SPI2_MISO: now reaches U6.27 (PB14)
- net SPI2_MISO: now also U5.24 (SDA/SDI)
- net SPI2_MOSI: now reaches U6.28 (PB15)
- net SPI2_MOSI: now also U5.9 (SDO/AD0)
- net IMU_INT: now reaches U6.29 (PA8)
- net IMU_INT: now also U5.12 (INT1)
- net INT1: no longer names the net of U6.21 (PB10)
- net INT1: no longer U5.12 (INT1)
- net SPI1_CS0 renamed SPI1_CS
- net SPI1_CS1: no longer names the net of U6.20 (PB2)
- net SPI1_CS1: no longer U5.22 (~{CS})
- removed net VREG_O: C7.1, FB1.1, U3.2 (VO)
- new net: C4.1, FB1.2, U3.3 (VI)
- new net CONN_D+: J1.A6 (D+), J1.B6 (D+), U2.3 (I/O2)
- new net CONN_D-: J1.A7 (D-), J1.B7 (D-), U2.1 (I/O1)
- no-connect marks 5 -> 24
Other:
- moved on the sheet: C4, C7, FB1, R4, R5, U3

Commit message: Add files via upload
Parts:
- U6: footprint Package_DFN_QFN:QFN-48-1EP_7x7mm_P0.5mm_EP5.15x5.15mm_ThermalVias -> Package_DFN_QFN:QFN-48-1EP_7x7mm_P0.5mm_EP5.15x5.15mm
Changed lines of the file:
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@@
 			)
 		)
-		(property "Footprint" "Package_DFN_QFN:QFN-48-1EP_7x7mm_P0.5mm_EP5.15x5.15mm_ThermalVias"
+		(property "Footprint" "Package_DFN_QFN:QFN-48-1EP_7x7mm_P0.5mm_EP5.15x5.15mm"
 			(at 276.86 119.38 0)
 			(effects

Commit message: Add files via upload
Parts:
- U6: footprint Package_DFN_QFN:QFN-48-1EP_7x7mm_P0.5mm_EP5.15x5.15mm -> Package_DFN_QFN:QFN-48-1EP_7x7mm_P0.5mm_EP5.15x5.15mm_ThermalVias
Changed lines of the file:
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@@
 			)
 		)
-		(property "Footprint" "Package_DFN_QFN:QFN-48-1EP_7x7mm_P0.5mm_EP5.15x5.15mm"
+		(property "Footprint" "Package_DFN_QFN:QFN-48-1EP_7x7mm_P0.5mm_EP5.15x5.15mm_ThermalVias"
 			(at 276.86 119.38 0)
 			(effects
